File: KiCAD/smart-proofing-box/host.kicad_sch (KiCad schematic)
At the start: 21 parts, among them SW2 SW_Push, U1 ESP32-C3, Y1 40MHz

Commit message: continued sketching rough design
Parts:
- added C17: 100n, Capacitor_SMD:C_0402_1005Metric_Pad0.74x0.62mm_HandSolder, symbol Device:C
- added U2: ZD25WQ32C, Package_SO:SOP-8_5.28x5.23mm_P1.27mm, symbol Prj_Memory_Flash:ZD25WQ32C
Connections:
- net +3.3V: now also C17.1, U2.8 (VCC)
- net GND: now also C17.2, U2.4 (GND)
- net MOSI: now reaches U1.10 (MTDI)
- net SS: now reaches U1.12 (MTCK)
- net MISO: now reaches U1.13 (MTDO)
- net I2C_SDA: now reaches U1.14 (GPIO8)
- net I2C_SCL: now reaches U1.16 (GPIO10)
- net SPIHD: now reaches U1.19 (SPIHD)
- net SPIHD: now also U2.7 (~{HOLD}/IO3)
- net SPIWP: now reaches U1.20 (SPIWP)
- net SPIWP: now also U2.3 (~{WP}/IO2)
- net SPCS0: now reaches U1.21 (SPICS0)
- net SPCS0: now also U2.1 (~{CS})
- net SPICLK: now reaches U1.22 (SPICLK)
- net SPICLK: now also U2.6 (SCK)
- net SPID: now reaches U1.23 (SPID)
- net SPID: now also U2.5 (SI/IO0)
- net SPIQ: now reaches U1.24 (SPIQ)
- net SPIQ: now also U2.2 (SO/IO1)
- net IO_INT: now reaches U1.27 (U0RXD)
- net Signal: now reaches U1.28 (U0TXD)
- net Sensor_T_Box: now reaches U1.4 (XTAL_32K_P)
- net Sensor_T_Inside: now reaches U1.5 (XTAL_32K_N)
- net Sensor_T_Outside: now reaches U1.6 (GPIO2)
- net FAN: now reaches U1.8 (GPIO3)
- net SCK: now reaches U1.9 (MTMS)
Other:
- moved on the sheet: AE1, C5, C6, C7, L1, R5, SW2

Commit message: continued work on schematic
Connections:
- net +3.3V renamed +3V3
- net FAN: no longer names the net of U1.8 (GPIO3)
- net Signal: no longer names the net of U1.28 (U0TXD)
Other:
- moved on the sheet: C10, C11, C12, C13, C14, C15, C17, C8, C9, L2, U2
