File: KiCAD/smart-proofing-box/peltier.kicad_sch (KiCad schematic)
At the start: 0 parts

Commit message: continued sketching rough design
Changed lines of the file:
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@@
 	(paper "A4")
 	(hierarchical_label "Polarity"
-		(shape input)
+		(shape output)
 		(at 55.88 69.85 0)
 		(fields_autoplaced yes)
@@
 		)
 	)
-	(hierarchical_label "Sensor"
+	(hierarchical_label "FAN"
 		(shape output)
-		(at 55.88 72.39 0)
+		(at 55.88 74.93 0)
+		(fields_autoplaced yes)
+		(effects
+			(font
+				(size 1.27 1.27)
+			)
+			(justify left)
+		)
+	)
+	(hierarchical_label "Sensor_T_Box"
+		(shape input)
+		(at 59.69 85.09 0)
+		(fields_autoplaced yes)
+		(effects
+			(font
+				(size 1.27 1.27)
+			)
+			(justify left)
+		)
+	)
+	(hierarchical_label "Sensor_T_Outside"
+		(shape input)
+		(at 59.69 90.17 0)
+		(fields_autoplaced yes)
+		(effects
+			(font
+				(size 1.27 1.27)
+			)
+			(justify left)
+		)
+	)
+	(hierarchical_label "Sensor_T_Inside"
+		(shape input)
+		(at 59.69 87.63 0)
 		(fields_autoplaced yes)
 		(effects
@@
 	)
 	(hierarchical_label "Signal"
-		(shape input)
+		(shape output)
 		(at 55.88 66.04 0)
 		(fields_autoplaced yes)

Commit message: continued work on schematic
Changed lines of the file:
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@@
 	(generator_version "8.0")
 	(paper "A4")
+	(hierarchical_label "FAN_Outside"
+		(shape output)
+		(at 55.88 77.47 0)
+		(fields_autoplaced yes)
+		(effects
+			(font
+				(size 1.27 1.27)
+			)
+			(justify left)
+		)
+	)
 	(hierarchical_label "Polarity"
 		(shape output)
@@
 		)
 	)
-	(hierarchical_label "FAN"
+	(hierarchical_label "FAN_Inside"
 		(shape output)
 		(at 55.88 74.93 0)
